Commit message: work about the controller of the sim drone

File: src/sim_drone/config/main.urdf.xacro (robot description, xacro)
@@ -1,11 +1,21 @@
 <?xml version="1.0"?>
-<robot name="sim_drone" xmlns:xacro="http://www.ros.org/wiki/xacro">
+<robot xmlns:xacro="http://www.ros.org/wiki/xacro" name="sim_drone">
     <!-- Include the robot and gazebo configurations -->
     <xacro:include filename="$(find sim_drone)/config/my_robot.urdf.xacro"/>
-    <!-- Main properties can be defined here if needed -->
-    <xacro:property name="mesh_scale" value="0.008" />
-    <xacro:property name="propeller_mass" value="0.05" />
-    <xacro:property name="base_mass" value="0.15" />
-    <!-- Ensure correct collision shape -->
-    <xacro:property name="collision_mesh" value="package://urdf/WholeDrone_collision.STL" />
+    <xacro:include filename="$(find sim_drone)/config/motor.ros2_control.xacro"/>
+    <!-- Main properties -->
+    <xacro:property name="mesh_scale" value="0.008"/>
+    <xacro:property name="propeller_mass" value="0.05"/>
+    <xacro:property name="base_mass" value="0.15"/>
+    <!-- Collision mesh -->
+    <xacro:property name="collision_mesh" value="package://urdf/WholeDrone_collision.STL"/>
+    <!-- Add ros2_control configuration -->
+    <xacro:drone_ros2_control name="DroneControl"/>
+    <!-- Add gazebo_ros2_control plugin -->
+    <gazebo>
+        <plugin filename="libgazebo_ros2_control.so" name="gazebo_ros2_control">
+            <parameters>$(find sim_drone)/config/controller_config.yaml</parameters>
+            <robot_sim_type>gazebo_ros2_control/GazeboSystem</robot_sim_type>
+        </plugin>
+    </gazebo>
 </robot>
