Commit message: fix the inertia and the collsiion

File: install/ground_bot/share/ground_bot/urdf/robot_description.urdf (robot description, URDF)
Before this commit: robot hamma_bot, 11 links, 10 joints
Links:
- link wheel_fl: mass None -> 1; geometry collision cylinder length=0.1 radius=0.28; visual cylinder length=0.1 radius=0.28
- link wheel_fr: mass None -> 1; geometry collision cylinder length=0.1 radius=0.28; visual cylinder length=0.1 radius=0.28
- link wheel_rl: mass None -> 1; geometry collision cylinder length=0.1 radius=0.28; visual cylinder length=0.1 radius=0.28
- link wheel_rr: mass None -> 1; geometry collision cylinder length=0.1 radius=0.28; visual cylinder length=0.1 radius=0.28

Commit message: finish build the ackeramn bot for the hamma

File: install/ground_bot/share/ground_bot/urdf/robot_description.urdf (robot description, URDF)
Before this commit: robot hamma_bot, 11 links, 10 joints
Links:
- link steer_link_fl: mass None -> 0.1
- link steer_link_fr: mass None -> 0.1

Commit message: start to build the nav_bringup

File: install/ground_bot/share/ground_bot/urdf/robot_description.urdf (robot description, URDF)
Before this commit: robot hamma_bot, 11 links, 10 joints
Links:
- removed link camera
- removed link imu
- removed link lidar
- added link camera_frame
- added link camera_link; visual box size=0.2 0.6 0.2
- added link imu_link; visual box size=0.4 0.4 0.3
- added link lidar_link; visual cylinder length=0.1 radius=0.3
Joints:
- removed joint base_link_to_camera
- added joint camera_frame_joint: type fixed, parent camera_link, child camera_frame, origin xyz=0 0 0 rpy=0 0 0
- added joint camera_joint: type fixed, parent base_link, child camera_link, origin xyz=1.6 0 0.4 rpy=0 0 0
- joint base_link_to_imu: child imu -> imu_link
- joint base_link_to_lidar: child lidar -> lidar_link

Commit message: add somthing for my work

File: install/ground_bot/share/ground_bot/urdf/robot_description.urdf (robot description, URDF)
Before this commit: robot hamma_bot, 12 links, 11 joints
Links:
- removed link camera_link
- added link camera_link_left; visual box size=0.2 0.6 0.2
- added link camera_link_right; visual box size=0.2 0.6 0.2
- link camera_frame: geometry visual box size=0.2 0.2 0.2
Joints:
- removed joint camera_frame_joint
- removed joint camera_joint
- added joint base_link_to_camera_frame: type fixed, parent base_link, child camera_frame, origin xyz=1.6 0 0.4 rpy=0 0 0
- added joint camera_joint_left: type fixed, parent base_link, child camera_link_left, origin xyz=1.6 0 0.4 rpy=0 0 -1.5708
- added joint camera_joint_right: type fixed, parent base_link, child camera_link_right, origin xyz=1.6 0 0.4 rpy=0 0 1.5708

Commit message: start of the work day

File: install/ground_bot/share/ground_bot/urdf/robot_description.urdf (robot description, URDF)
Before this commit: robot hamma_bot, 13 links, 12 joints
Links:
- removed link world_link
- added link base_footprint, mass 0
Joints:
- joint base_joint: parent world_link -> base_footprint

Commit message: naor fix the odom part

File: install/ground_bot/share/ground_bot/urdf/robot_description.urdf (robot description, URDF)
Before this commit: robot hamma_bot, 13 links, 12 joints
Links:
- link base_footprint: mass 0 -> None
Joints:
- joint base_joint: origin xyz=0 0 0.5 rpy=0 0 0 -> xyz=0.0 0.0 0.0 rpy=0 0 0

Commit message: not work yet

File: install/ground_bot/share/ground_bot/urdf/robot_description.urdf (robot description, URDF)
Before this commit: robot hamma_bot, 13 links, 12 joints
Links:
- added link camera_front_link; visual box size=0.07 0.07 0.03
Joints:
- added joint camera_top_joint: type fixed, parent base_link, child camera_front_link, origin xyz=1.9 0 0.3 rpy=0 0 0
- joint base_joint: origin xyz=0.0 0.0 0.0 rpy=0 0 0 -> xyz=0.0 0.0 1.0 rpy=0 0 0

Commit message: almost finish the slam toolbox

File: install/ground_bot/share/ground_bot/urdf/robot_description.urdf (robot description, URDF)
Before this commit: robot hamma_bot, 13 links, 12 joints
Links:
- link lidar_link: geometry visual box size=0.1 0.1 0.1
Joints:
- joint base_link_to_lidar: origin xyz=0 0 0.25 rpy=0 0 0 -> xyz=1.88 0 -0.15 rpy=0 0 0
- joint front_left_wheel_joint: axis 0 0 1 -> 0 0 -1
- joint front_right_wheel_joint: axis 0 0 1 -> 0 0 -1
- joint rear_left_wheel_joint: axis 0 0 1 -> 0 0 -1
- joint rear_right_wheel_joint: axis 0 0 1 -> 0 0 -1
