Commit message: fix robot oroitation

File: install/ground_bot/share/ground_bot/urdf/ground_bot_descriptor.urdf (robot description, URDF)
Before this commit: robot ground_bot, 8 links, 7 joints
Links:
- link base_link: mass 10 -> 100
Joints:
- removed joint base_footprint_joint
- added joint base_joint: type fixed, parent base_link, child base_footprint, origin xyz=0.0 0.0 -0.15 rpy=0 0 0
- joint wheel_left_joint: axis 0 0 1 -> 0 0 -1; origin xyz=-0.15 -0.153 -0.02 rpy=1.577 0 0 -> xyz=-0.15 0.18 -0.02 rpy=1.577 0 0
- joint wheel_right_joint: axis 0 0 1 -> 0 0 -1; origin xyz=-0.15 0.153 -0.02 rpy=1.577 0 0 -> xyz=-0.15 -0.18 -0.02 rpy=1.577 0 0

Commit message: almost finish the integration of the realsense camera

File: install/ground_bot/share/ground_bot/urdf/ground_bot_descriptor.urdf (robot description, URDF)
Before this commit: robot ground_bot, 8 links, 7 joints
Links:
- added link depth_camera_real_link; visual box size=0.01 0.01 0.01
- added link lidar_link; visual box size=0.01 0.01 0.01
- link caster_wheel_link: mass 10 -> 30
Joints:
- added joint depth_camera_real_joint: type fixed, parent base_link, child depth_camera_real_link, origin xyz=0.2 0 0.04 rpy=0 0 0
- added joint lidar_joint: type fixed, parent base_link, child lidar_link, origin xyz=0.2 0 0.03 rpy=0 0 0

Commit message: finish the realsesnes

File: install/ground_bot/share/ground_bot/urdf/ground_bot_descriptor.urdf (robot description, URDF)
Before this commit: robot ground_bot, 10 links, 9 joints
Links:
- removed link depth_camera_real_link
- added link camera_link; visual box size=0.01 0.01 0.01
Joints:
- removed joint depth_camera_real_joint
- added joint camera_mount_joint: type fixed, parent base_link, child camera_link, origin xyz=0.2 0 0.04 rpy=0 1.57 0

Commit message: fix

File: install/ground_bot/share/ground_bot/urdf/ground_bot_descriptor.urdf (robot description, URDF)
Before this commit: robot ground_bot, 10 links, 9 joints
Links:
- link launch_pad_link: mass None -> 10; geometry collision cylinder length=0.02 radius=0.15; visual cylinder length=0.02 radius=0.15
- link stand_link: mass None -> 10; geometry collision cylinder length=0.2 radius=0.01; visual cylinder length=0.2 radius=0.01

Commit message: fix the map

File: install/ground_bot/share/ground_bot/urdf/ground_bot_descriptor.urdf (robot description, URDF)
Before this commit: robot ground_bot, 10 links, 9 joints
Links:
- removed link camera_link
- link lidar_link: mass None -> 0.125; geometry collision cylinder length=0.055 radius=0.0508; visual cylinder length=0.01 radius=0.01
Joints:
- removed joint camera_mount_joint
- joint lidar_joint: origin xyz=0.2 0 0.03 rpy=0 0 0 -> xyz=0.2 0 0.04 rpy=0 0 0
