Commit message: at this state the urdf of the swing drone lock fine

File: src/robot_description/urdf/motor.ros2_control.xacro (robot description, xacro)
@@ -4,5 +4,7 @@
         <ros2_control name="${name}" type="system">
             <hardware>
-                <plugin>ign_ros2_control/IgnitionSystem</plugin>
+                <plugin>gz_ros2_control/GzSystem</plugin>
+                <param name="world_name">motor_physics_test</param>
+                <param name="robot_param">robot_description</param>
             </hardware>
             <!-- Front Right Propeller -->
@@ -46,17 +48,4 @@
                 <state_interface name="effort"/>
             </joint>
-            <!-- IMU Sensor -->
-            <sensor name="imu_sensor">
-                <state_interface name="orientation.x"/>
-                <state_interface name="orientation.y"/>
-                <state_interface name="orientation.z"/>
-                <state_interface name="orientation.w"/>
-                <state_interface name="angular_velocity.x"/>
-                <state_interface name="angular_velocity.y"/>
-                <state_interface name="angular_velocity.z"/>
-                <state_interface name="linear_acceleration.x"/>
-                <state_interface name="linear_acceleration.y"/>
-                <state_interface name="linear_acceleration.z"/>
-            </sensor>
         </ros2_control>
     </xacro:macro>

File: src/robot_description/urdf/my_robot.urdf.xacro (robot description, xacro)
@@ -10,5 +10,5 @@
         <visual>
             <geometry>
-                <mesh filename="file://robot_description/meshes/WholeDrone.STL" scale="0.008 0.008 0.008"/>
+                <mesh filename="package://robot_description/meshes/WholeDrone.STL" scale="0.008 0.008 0.008"/>
             </geometry>
             <origin xyz="0.56 -0.8275 -0.425" rpy="${pi/2} 0 ${pi}" />
@@ -34,5 +34,5 @@
             <visual>
                 <geometry>
-                    <mesh filename="file://robot_description/meshes/PropellerForRos.STL" scale="0.008 0.008 0.008"/>
+                    <mesh filename="package://robot_description/meshes/PropellerForRos.STL" scale="0.008 0.008 0.008"/>
                 </geometry>
                 <origin xyz="-0.269 0.3874 -0.2" rpy="${pi/2} 0 0" />
@@ -88,29 +88,3 @@
         <dynamics damping="0.01" friction="0.01"/>
     </joint>
-    <!-- IMU Link -->
-    <link name="imu_link">
-        <visual>
-            <geometry>
-                <box size="0.02 0.02 0.02"/>
-            </geometry>
-            <material name="blue"/>
-        </visual>
-        <collision>
-            <geometry>
-                <box size="0.02 0.02 0.02"/>
-            </geometry>
-        </collision>
-        <inertial>
-            <mass value="0.01"/>
-            <inertia ixx="0.0001" ixy="0" ixz="0"
-                    iyy="0.0001" iyz="0"
-                    izz="0.0001"/>
-        </inertial>
-    </link>
-    <!-- IMU Joint -->
-    <joint name="imu_joint" type="fixed">
-        <parent link="base_link"/>
-        <child link="imu_link"/>
-        <origin xyz="0 0 0" rpy="0 0 0"/>
-    </joint>
 </robot>

File: src/robot_description/urdf/robot_gazebo.xacro (robot description, xacro)
@@ -3,5 +3,5 @@
     <!-- Gazebo Control Plugin -->
     <gazebo>
-        <plugin filename="gz-sim-multicopter-control-system" name="ignition::gazebo::systems::MulticopterVelocityControl">
+        <plugin filename="gz-sim-multicopter-control-system" name="gz::sim::systems::MulticopterVelocityControl">
             <robotNamespace>sim_drone</robotNamespace>
             <commandSubTopic>cmd_vel</commandSubTopic>
@@ -46,24 +46,69 @@
         </plugin>
     </gazebo>
-    <gazebo reference="imu_link">
-        <gravity>true</gravity>
-        <sensor name="imu_sensor" type="imu">
-        <always_on>true</always_on>
-        <update_rate>100</update_rate>
-        <visualize>true</visualize>
-        <topic>/imu/data</topic>
-        <plugin filename="ignition-gazebo-imu-system"
-                    name="ignition::gazebo::systems::Imu">
-            <bodyName>imu_link</bodyName>
-            <updateRateHZ>100.0</updateRateHZ>
-            <gaussianNoise>0.01</gaussianNoise>
-            <xyzOffset>0 0 0</xyzOffset>
-            <rpyOffset>0 0 0</rpyOffset>
-            <frameName>imu_link</frameName>
-            <initialOrientationAsReference>false</initialOrientationAsReference>
-        </plugin>
-        <pose>0 0 0 0 0 0</pose>
-        </sensor>
-    </gazebo>
+  <gazebo reference="imu_link">
+    <sensor name="imu_sensor" type="imu">
+      <ignition_frame_id>imu_link</ignition_frame_id>
+      <plugin filename="ignition-gazebo-imu-system" name="ignition::gazebo::systems::Imu">
+      </plugin>
+      <topic>imu</topic>
+      <always_on>true</always_on>
+      <update_rate>100</update_rate>
+      <visualize>true</visualize>
+      <imu>
+        <angular_velocity>
+          <x>
+            <noise type="gaussian">
+              <mean>0.0</mean>
+              <stddev>2e-4</stddev>
+              <bias_mean>0.0000075</bias_mean>
+              <bias_stddev>0.0000008</bias_stddev>
+            </noise>
+          </x>
+          <y>
+            <noise type="gaussian">
+              <mean>0.0</mean>
+              <stddev>2e-4</stddev>
+              <bias_mean>0.0000075</bias_mean>
+              <bias_stddev>0.0000008</bias_stddev>
+            </noise>
+          </y>
+          <z>
+            <noise type="gaussian">
+              <mean>0.0</mean>
+              <stddev>2e-4</stddev>
+              <bias_mean>0.0000075</bias_mean>
+              <bias_stddev>0.0000008</bias_stddev>
+            </noise>
+          </z>
+        </angular_velocity>
+        <linear_acceleration>
+          <x>
+            <noise type="gaussian">
+              <mean>0.0</mean>
+              <stddev>1.7e-2</stddev>
+              <bias_mean>0.1</bias_mean>
+              <bias_stddev>0.001</bias_stddev>
+            </noise>
+          </x>
+          <y>
+            <noise type="gaussian">
+              <mean>0.0</mean>
+              <stddev>1.7e-2</stddev>
+              <bias_mean>0.1</bias_mean>
+              <bias_stddev>0.001</bias_stddev>
+            </noise>
+          </y>
+          <z>
+            <noise type="gaussian">
+              <mean>0.0</mean>
+              <stddev>1.7e-2</stddev>
+              <bias_mean>0.1</bias_mean>
+              <bias_stddev>0.001</bias_stddev>
+            </noise>
+          </z>
+        </linear_acceleration>
+      </imu>
+    </sensor>
+  </gazebo>
     <!-- Gazebo Colors -->
     <gazebo reference="base_link"><material>Gazebo/White</material></gazebo>
