Commit message: push for raz

File: src/swing_drone/urdf/main.urdf.xacro (robot description, xacro)
@@ -4,3 +4,5 @@
     <xacro:include filename="$(find swing_drone)/urdf/robot_gazebo.urdf.xacro"/>
     <xacro:include filename="$(find swing_drone)/urdf/robot_control.urdf.xacro"/>
+    <!-- Call the control macro to instantiate ros2_control -->
+    <xacro:swing_drone_control name="drone_controler"/>
 </robot>

File: src/swing_drone/urdf/robot_control.urdf.xacro (robot description, xacro)
@@ -8,41 +8,49 @@
             <joint name="A_prop_joint">
                 <command_interface name="effort"></command_interface>
+                <state_interface name="position"/>
+                <state_interface name="velocity"/>
                 <state_interface name="effort"/>
-                <state_interface name="velocity"/>
             </joint>
             <joint name="B_prop_joint">
                 <command_interface name="effort"></command_interface>
+                <state_interface name="position"/>
+                <state_interface name="velocity"/>
                 <state_interface name="effort"/>
-                <state_interface name="velocity"/>
             </joint>
             <joint name="C_prop_joint">
                 <command_interface name="effort"></command_interface>
+                <state_interface name="position"/>
+                <state_interface name="velocity"/>
                 <state_interface name="effort"/>
-                <state_interface name="velocity"/>
             </joint>
             <joint name="D_prop_joint">
                 <command_interface name="effort"></command_interface>
+                <state_interface name="position"/>
+                <state_interface name="velocity"/>
                 <state_interface name="effort"/>
-                <state_interface name="velocity"/>
             </joint>
             <joint name="E_prop_joint">
                 <command_interface name="effort"></command_interface>
+                <state_interface name="position"/>
+                <state_interface name="velocity"/>
                 <state_interface name="effort"/>
-                <state_interface name="velocity"/>
             </joint>
             <joint name="F_prop_joint">
                 <command_interface name="effort"></command_interface>
+                <state_interface name="position"/>
+                <state_interface name="velocity"/>
                 <state_interface name="effort"/>
-                <state_interface name="velocity"/>
             </joint>
             <joint name="G_prop_joint">
                 <command_interface name="effort"></command_interface>
+                <state_interface name="position"/>
+                <state_interface name="velocity"/>
                 <state_interface name="effort"/>
-                <state_interface name="velocity"/>
             </joint>
             <joint name="H_prop_joint">
                 <command_interface name="effort"></command_interface>
+                <state_interface name="position"/>
+                <state_interface name="velocity"/>
                 <state_interface name="effort"/>
-                <state_interface name="velocity"/>
             </joint>
         </ros2_control>
@@ -50,5 +58,5 @@
             <plugin filename="ign_ros2_control-system" name="ign_ros2_control::IgnitionROS2ControlPlugin">
                 <robot_param_node>robot_state_publisher</robot_param_node>
-                <!-- <parameters>$(find swing_drone)/config/my_controllers.yaml</parameters> -->
+                <parameters>$(find swing_drone)/config/drone_controller.yaml</parameters>
             </plugin>
         </gazebo>

File: src/swing_drone/urdf/robot_description.urdf.xacro (robot description, xacro)
@@ -1,4 +1,14 @@
 <?xml version="1.0"?>
 <robot name="swing_drone" xmlns:xacro="http://www.ros.org/wiki/xacro">
+  <!-- Dummy map link as root to avoid KDL parser warning -->
+  <link name="map">
+    <!-- No inertia for dummy root link -->
+  </link>
+  <!-- Fixed joint connecting map to base_link -->
+  <joint name="map_to_base" type="fixed">
+    <parent link="map"/>
+    <child link="base_link"/>
+    <origin xyz="0 0 0" rpy="0 0 0"/>
+  </joint>
   <link
     name="base_link">

File: src/swing_drone/urdf/robot_gazebo.urdf.xacro (robot description, xacro)
@@ -1,4 +1,10 @@
 <?xml version="1.0"?>
 <robot xmlns:xacro="http://www.ros.org/wiki/xacro" name="swing_drone">
+    <gazebo>
+        <plugin filename="ign_ros2_control-system" name="ign_ros2_control::IgnitionROS2ControlPlugin">
+              <robot_param_node>robot_state_publisher</robot_param_node>
+              <parameters>$(find swing_drone)/config/drone_controller.yaml</parameters>
+        </plugin>
+    </gazebo>
     <gazebo>
         <plugin name='ignition::gazebo::systems::Physics' filename='ignition-gazebo-physics-system'/>
@@ -21,5 +27,5 @@
     <kp>1000000.0</kp>
     <kd>1.0</kd>
-    <selfCollide>false</selfCollide>
+    <selfCollide>true</selfCollide>
   </gazebo>
   <gazebo reference="fr_link">
