Commit message: the gazebo almost work

File: src/swing_drone/urdf/robot_description.urdf.xacro (robot description, xacro)
@@ -1,7 +1,6 @@
-<?xml version="1.0" encoding="utf-8"?>
-<robot
-  name="swing_drone">
-  <link
-    name="base_link ">
+<?xml version="1.0"?>
+<robot name="swing_drone" xmlns:xacro="http://www.ros.org/wiki/xacro">
+  <link
+    name="base_link">
     <inertial>
       <origin
@@ -43,4 +42,43 @@
   </link>
   <link
+    name="imu_link">
+    <inertial>
+      <origin xyz="0 0 0" rpy="0 0 0"/>
+      <mass value="0.001"/>
+      <inertia ixx="1e-6" ixy="0" ixz="0" iyy="1e-6" iyz="0" izz="1e-6"/>
+    </inertial>
+    <visual>
+      <origin
+        xyz="0 0 0"
+        rpy="0 0 0" />
+      <geometry>
+        <box
+          size="0.01 0.01 0.01" />
+      </geometry>
+    </visual>
+    <collision>
+      <origin
+        xyz="0 0 0"
+        rpy="0 0 0" />
+      <geometry>
+        <box
+          size="0.01 0.01 0.01" />
+      </geometry>
+    </collision>
+  </link>
+  <joint
+    name="imu_joint"
+    type="fixed">
+    <parent
+      link="base_link" />
+    <child
+      link="imu_link" />
+    <origin
+      xyz="0 0 0"
+      rpy="0 0 0" />
+    <axis
+      xyz="0 0 1" />
+  </joint>
+  <link
     name="fr_link">
     <inertial>
@@ -64,5 +102,5 @@
       <geometry>
         <mesh
-          filename="package://swing_drone/meshes/fr_link.STL" />
+          filename="package://swing_drone/meshes/arm.STL" />
       </geometry>
       <material
@@ -78,5 +116,5 @@
       <geometry>
         <mesh
-          filename="package://swing_drone/meshes/fr_link.STL" />
+          filename="package://swing_drone/meshes/arm.STL" />
       </geometry>
     </collision>
@@ -89,5 +127,5 @@
       rpy="1.5708 0 2.3562" />
     <parent
-      link="base_link " />
+      link="base_link" />
     <child
       link="fr_link" />
@@ -117,5 +155,5 @@
       <geometry>
         <mesh
-          filename="package://swing_drone/meshes/A_prop_link.STL" />
+          filename="package://swing_drone/meshes/CCW_prop.STL" />
       </geometry>
       <material
@@ -131,5 +169,5 @@
       <geometry>
         <mesh
-          filename="package://swing_drone/meshes/A_prop_link.STL" />
+          filename="package://swing_drone/meshes/CCW_prop.STL" />
       </geometry>
     </collision>
@@ -170,5 +208,5 @@
       <geometry>
         <mesh
-          filename="package://swing_drone/meshes/B_prop_link.STL" />
+          filename="package://swing_drone/meshes/CW_prop.STL" />
       </geometry>
       <material
@@ -184,5 +222,5 @@
       <geometry>
         <mesh
-          filename="package://swing_drone/meshes/B_prop_link.STL" />
+          filename="package://swing_drone/meshes/CW_prop.STL" />
       </geometry>
     </collision>
@@ -223,5 +261,5 @@
       <geometry>
         <mesh
-          filename="package://swing_drone/meshes/br_link.STL" />
+          filename="package://swing_drone/meshes/arm.STL" />
       </geometry>
       <material
@@ -237,5 +275,5 @@
       <geometry>
         <mesh
-          filename="package://swing_drone/meshes/br_link.STL" />
+          filename="package://swing_drone/meshes/arm.STL" />
       </geometry>
     </collision>
@@ -248,5 +286,5 @@
       rpy="1.5707963267949 0 0.785398163397444" />
     <parent
-      link="base_link " />
+      link="base_link" />
     <child
       link="br_link" />
@@ -276,5 +314,5 @@
       <geometry>
         <mesh
-          filename="package://swing_drone/meshes/C_prop_link.STL" />
+          filename="package://swing_drone/meshes/CCW_prop.STL" />
       </geometry>
       <material
@@ -290,5 +328,5 @@
       <geometry>
         <mesh
-          filename="package://swing_drone/meshes/C_prop_link.STL" />
+          filename="package://swing_drone/meshes/CCW_prop.STL" />
       </geometry>
     </collision>
@@ -329,5 +367,5 @@
       <geometry>
         <mesh
-          filename="package://swing_drone/meshes/D_prop_link.STL" />
+          filename="package://swing_drone/meshes/CW_prop.STL" />
       </geometry>
       <material
@@ -343,5 +381,5 @@
       <geometry>
         <mesh
-          filename="package://swing_drone/meshes/D_prop_link.STL" />
+          filename="package://swing_drone/meshes/CW_prop.STL" />
       </geometry>
     </collision>
@@ -382,5 +420,5 @@
       <geometry>
         <mesh
-          filename="package://swing_drone/meshes/bl_link.STL" />
+          filename="package://swing_drone/meshes/arm.STL" />
       </geometry>
       <material
@@ -396,5 +434,5 @@
       <geometry>
         <mesh
-          filename="package://swing_drone/meshes/bl_link.STL" />
+          filename="package://swing_drone/meshes/arm.STL" />
       </geometry>
     </collision>
@@ -407,5 +445,5 @@
       rpy="1.5707963267949 0 -0.785398163397454" />
     <parent
-      link="base_link " />
+      link="base_link" />
     <child
       link="bl_link" />
@@ -435,5 +473,5 @@
       <geometry>
         <mesh
-          filename="package://swing_drone/meshes/E_prop_link.STL" />
+          filename="package://swing_drone/meshes/CCW_prop.STL" />
       </geometry>
       <material
@@ -449,5 +487,5 @@
       <geometry>
         <mesh
-          filename="package://swing_drone/meshes/E_prop_link.STL" />
+          filename="package://swing_drone/meshes/CCW_prop.STL" />
       </geometry>
     </collision>
@@ -488,5 +526,5 @@
       <geometry>
         <mesh
-          filename="package://swing_drone/meshes/F_prop_link.STL" />
+          filename="package://swing_drone/meshes/CW_prop.STL" />
       </geometry>
       <material
@@ -502,5 +540,5 @@
       <geometry>
         <mesh
-          filename="package://swing_drone/meshes/F_prop_link.STL" />
+          filename="package://swing_drone/meshes/CW_prop.STL" />
       </geometry>
     </collision>
@@ -541,5 +579,5 @@
       <geometry>
         <mesh
-          filename="package://swing_drone/meshes/fl_link.STL" />
+          filename="package://swing_drone/meshes/arm.STL" />
       </geometry>
       <material
@@ -555,5 +593,5 @@
       <geometry>
         <mesh
-          filename="package://swing_drone/meshes/fl_link.STL" />
+          filename="package://swing_drone/meshes/arm.STL" />
       </geometry>
     </collision>
@@ -566,5 +604,5 @@
       rpy="1.5707963267949 0 -2.35619449019234" />
     <parent
-      link="base_link " />
+      link="base_link" />
     <child
       link="fl_link" />
@@ -594,5 +632,5 @@
       <geometry>
         <mesh
-          filename="package://swing_drone/meshes/G_prop_link.STL" />
+          filename="package://swing_drone/meshes/CCW_prop.STL" />
       </geometry>
       <material
@@ -608,5 +646,5 @@
       <geometry>
         <mesh
-          filename="package://swing_drone/meshes/G_prop_link.STL" />
+          filename="package://swing_drone/meshes/CCW_prop.STL" />
       </geometry>
     </collision>
@@ -647,5 +685,5 @@
       <geometry>
         <mesh
-          filename="package://swing_drone/meshes/H_prop_link.STL" />
+          filename="package://swing_drone/meshes/CW_prop.STL" />
       </geometry>
       <material
@@ -661,5 +699,5 @@
       <geometry>
         <mesh
-          filename="package://swing_drone/meshes/H_prop_link.STL" />
+          filename="package://swing_drone/meshes/CW_prop.STL" />
       </geometry>
     </collision>

Commit message: another test with raz

File: src/swing_drone/urdf/robot_description.urdf.xacro (robot description, xacro)
@@ -14,15 +14,15 @@
     <inertial>
       <origin
-        xyz="-9.81636642918719E-08 0.0306931155314605 6.86147954927806E-06"
-        rpy="0 0 0" />
-      <mass
-        value="0.489642795099214" />
-      <inertia
-        ixx="0.00550730711851782"
-        ixy="1.75918722866926E-09"
-        ixz="8.00407972816657E-09"
-        iyy="0.0106757497435687"
-        iyz="4.08917538783145E-08"
-        izz="0.00550715316059604" />
+        xyz="0 0.0307 0"
+        rpy="0 0 0" />
+      <mass
+        value="0.49" />
+      <inertia
+        ixx="0.0055"
+        ixy="0"
+        ixz="0"
+        iyy="0.01067"
+        iyz="0"
+        izz="0.0055" />
     </inertial>
     <visual>
@@ -84,15 +84,15 @@
     <inertial>
       <origin
-        xyz="5.72722553709436E-08 0.00838518201458534 -0.169743642048481"
-        rpy="0 0 0" />
-      <mass
-        value="0.0712984135491828" />
-      <inertia
-        ixx="1.25109623769764E-05"
-        ixy="-5.80866736119285E-11"
-        ixz="3.10377556603639E-11"
-        iyy="1.96234830559855E-05"
-        iyz="7.47360228967648E-12"
-        izz="1.31602072697672E-05" />
+        xyz="0 0.00839 -0.16975"
+        rpy="0 0 0" />
+      <mass
+        value="0.0713" />
+      <inertia
+        ixx="0.00001"
+        ixy="0"
+        ixz="0"
+        iyy="0.00001"
+        iyz="0"
+        izz="0.00001" />
     </inertial>
     <visual>
@@ -137,15 +137,15 @@
     <inertial>
       <origin
-        xyz="8.7159E-06 8.1377E-06 0.0069037"
+        xyz="0 0 0.0069037"
         rpy="0 0 0" />
       <mass
         value="0.0030458" />
       <inertia
-        ixx="1.0159E-06"
-        ixy="7.1666E-10"
-        ixz="-4.0698E-11"
-        iyy="1.017E-06"
-        iyz="-9.5763E-12"
-        izz="1.9885E-06" />
+        ixx="0.00001"
+        ixy="0"
+        ixz="0"
+        iyy="0.00001"
+        iyz="0"
+        izz="0.00001" />
     </inertial>
     <visual>
@@ -190,15 +190,15 @@
     <inertial>
       <origin
-        xyz="-2.9519E-06 6.6171E-06 0.0069036"
+        xyz="0 0 0.0069036"
         rpy="0 0 0" />
       <mass
         value="0.0030461" />
       <inertia
-        ixx="1.017E-06"
-        ixy="5.094E-10"
-        ixz="1.8144E-11"
-        iyy="1.0165E-06"
-        iyz="-2.7503E-11"
-        izz="1.989E-06" />
+        ixx="0.00001"
+        ixy="0"
+        ixz="0"
+        iyy="0.00001"
+        iyz="0"
+        izz="0.00001" />
     </inertial>
     <visual>
@@ -243,15 +243,15 @@
     <inertial>
       <origin
-        xyz="5.6967214640888E-08 0.00838518216887453 -0.169743641529002"
-        rpy="0 0 0" />
-      <mass
-        value="0.0712984116406711" />
-      <inertia
-        ixx="1.25109622044214E-05"
-        ixy="-5.80830005690429E-11"
-        ixz="3.10080125884296E-11"
-        iyy="1.96234829027007E-05"
-        iyz="7.49851524519673E-12"
-        izz="1.31602072915751E-05" />
+        xyz="0 0.00838518216887453 -0.169743641529002"
+        rpy="0 0 0" />
+      <mass
+        value="0.0713" />
+      <inertia
+        ixx="0.00001"
+        ixy="0"
+        ixz="0"
+        iyy="0.00001"
+        iyz="0"
+        izz="0.00001" />
     </inertial>
     <visual>
@@ -296,15 +296,15 @@
     <inertial>
       <origin
-        xyz="8.88376431135152E-06 8.24094770135453E-06 0.00690354838979317"
+        xyz="0 0 0.00690354838979317"
         rpy="0 0 0" />
       <mass
         value="0.00304576429500371" />
       <inertia
-        ixx="1.01583923908105E-06"
-        ixy="7.00300034386576E-10"
-        ixz="-4.34623235247216E-11"
-        iyy="1.01697553805106E-06"
-        iyz="-1.15132452923579E-11"
-        izz="1.98837107356726E-06" />
+        ixx="0.00001"
+        ixy="0"
+        ixz="0"
+        iyy="0.00001"
+        iyz="0"
+        izz="0.00001" />
     </inertial>
     <visual>
@@ -349,15 +349,15 @@
     <inertial>
       <origin
-        xyz="6.88758994921157E-06 -4.88396768444366E-07 0.0069035097240563"
+        xyz="0 0 0.0069035097240563"
         rpy="0 0 0" />
       <mass
         value="0.0030460170283791" />
       <inertia
-        ixx="1.01631129628996E-06"
-        ixy="-5.81174683431385E-11"
-        ixz="-3.79613417410503E-11"
-        iyy="1.01740859082528E-06"
-        iyz="3.60534564402912E-12"
-        izz="1.98927726106095E-06" />
+        ixx="0.00001"
+        ixy="0"
+        ixz="0"
+        iyy="0.00001"
+        iyz="0"
+        izz="0.00001" />
     </inertial>
     <visual>
@@ -402,15 +402,15 @@
     <inertial>
       <origin
-        xyz="5.57576253618631E-08 0.00838518201458557 -0.169743641788305"
-        rpy="0 0 0" />
-      <mass
-        value="0.0712984135491827" />
-      <inertia
-        ixx="1.25109623769764E-05"
-        ixy="-5.80805135568167E-11"
-        ixz="3.10377556599404E-11"
-        iyy="1.96234830559855E-05"
-        iyz="7.50888677807041E-12"
-        izz="1.31602072697672E-05" />
+        xyz="0 0.00838518201458557 -0.169743641788305"
+        rpy="0 0 0" />
+      <mass
+        value="0.0713" />
+      <inertia
+        ixx="0.00001"
+        ixy="0"
+        ixz="0"
+        iyy="0.00001"
+        iyz="0"
+        izz="0.00001" />
     </inertial>
     <visual>
@@ -455,15 +455,15 @@
     <inertial>
       <origin
-        xyz="2.7313275353727E-06 3.86682184189135E-07 0.00690385853098646"
+        xyz="0 0 0.00690385853098646"
         rpy="0 0 0" />
       <mass
         value="0.00304648811584682" />
       <inertia
-        ixx="1.01692766677989E-06"
-        ixy="-8.25590073897304E-12"
-        ixz="-2.9913999900015E-11"
-        iyy="1.01745813006253E-06"
-        iyz="1.47433389309506E-12"
-        izz="1.98993970966869E-06" />
+        ixx="0.00001"
+        ixy="0"
+        ixz="0"
+        iyy="0.00001"
+        iyz="0"
+        izz="0.00001" />
     </inertial>
     <visual>
@@ -508,15 +508,15 @@
     <inertial>
       <origin
-        xyz="-2.66120848305129E-06 6.72137493892833E-06 0.00690341554333757"
+        xyz="0 0 0.00690341554333757"
         rpy="0 0 0" />
       <mass
         value="0.00304581013536126" />
       <inertia
-        ixx="1.01706667134054E-06"
-        ixy="5.04989341627317E-10"
-        ixz="1.90640171727212E-11"
-        iyy="1.01648666014435E-06"
-        iyz="-2.22329153080792E-11"
-        izz="1.9891136648677E-06" />
+        ixx="0.00001"
+        ixy="0"
+        ixz="0"
+        iyy="0.00001"
+        iyz="0"
+        izz="0.00001" />
     </inertial>
     <visual>
@@ -561,15 +561,15 @@
     <inertial>
       <origin
-        xyz="5.77245295304477E-08 0.00838518205590654 -0.169743641875677"
-        rpy="0 0 0" />
-      <mass
-        value="0.0712984129705644" />
-      <inertia
-        ixx="1.25109623234441E-05"
-        ixy="-5.80860805952669E-11"
-        ixz="3.10312650412831E-11"
-        iyy="1.96234829906507E-05"
-        iyz="7.48087300370571E-12"
-        izz="1.31602072594632E-05" />
+        xyz="0 0.00838518205590654 -0.169743641875677"
+        rpy="0 0 0" />
+      <mass
+        value="0.0713" />
+      <inertia
+        ixx="0.00001"
+        ixy="0"
+        ixz="0"
+        iyy="0.00001"
+        iyz="0"
+        izz="0.00001" />
     </inertial>
     <visual>
@@ -614,15 +614,15 @@
     <inertial>
       <origin
-        xyz="3.62789022101406E-06 7.93861775136295E-06 0.00690342839194055"
+        xyz="0 0 0.00690342839194055"
         rpy="0 0 0" />
       <mass
         value="0.00304542470661797" />
       <inertia
-        ixx="1.01591118865216E-06"
-        ixy="7.11420493756258E-10"
-        ixz="-2.70428480861302E-11"
-        iyy="1.01623051835766E-06"
-        iyz="-1.42050794040357E-11"
-        izz="1.98769911974202E-06" />
+        ixx="0.00001"
+        ixy="0"
+        ixz="0"
+        iyy="0.00001"
+        iyz="0"
+        izz="0.00001" />
     </inertial>
     <visual>
@@ -667,15 +667,15 @@
     <inertial>
       <origin
-        xyz="-2.20600356380662E-06 4.87187253123134E-06 0.00690356262000323"
+        xyz="0 0 0.00690356262000323"
         rpy="0 0 0" />
       <mass
         value="0.00304597813849953" />
       <inertia
-        ixx="1.01676909541948E-06"
-        ixy="3.896174971715E-10"
-        ixz="1.6241830169863E-11"
-        iyy="1.01642948192595E-06"
-        iyz="-2.50490797824747E-11"
-        izz="1.98875407345364E-06" />
+        ixx="0.00001"
+        ixy="0"
+        ixz="0"
+        iyy="0.00001"
+        iyz="0"
+        izz="0.00001" />
     </inertial>
     <visual>

File: src/swing_drone/urdf/robot_gazebo.urdf.xacro (robot description, xacro)
@@ -7,3 +7,38 @@
         </plugin>
     </gazebo>
+    <gazebo reference="base_link">
+        <mu1>1.0</mu1>
+        <mu2>1.0</mu2>
+        <self_collide>1</self_collide>
+        <kp value="100000.0" />
+        <kd value="1.0" />
+    </gazebo>
+    <gazebo reference="fr_link  ">
+        <mu1>1.0</mu1>
+        <mu2>1.0</mu2>
+        <self_collide>1</self_collide>
+        <kp value="100000.0" />
+        <kd value="1.0" />
+    </gazebo>
+    <gazebo reference="fl_link">
+        <mu1>1.0</mu1>
+        <mu2>1.0</mu2>
+        <self_collide>1</self_collide>
+        <kp value="100000.0" />
+        <kd value="1.0" />
+    </gazebo>
+    <gazebo reference="br_link">
+        <mu1>1.0</mu1>
+        <mu2>1.0</mu2>
+        <self_collide>1</self_collide>
+        <kp value="100000.0" />
+        <kd value="1.0" />
+    </gazebo>
+    <gazebo reference="bl_link">
+        <mu1>1.0</mu1>
+        <mu2>1.0</mu2>
+        <self_collide>1</self_collide>
+        <kp value="100000.0" />
+        <kd value="1.0" />
+    </gazebo>
 </robot>
