Commit message: have problem with the gazebo - need fix it

File: src/swing_drone/urdf/robot_control.urdf.xacro (robot description, xacro)
@@ -55,10 +55,4 @@
             </joint>
         </ros2_control>
-        <gazebo>
-            <plugin filename="ign_ros2_control-system" name="ign_ros2_control::IgnitionROS2ControlPlugin">
-                <robot_param_node>robot_state_publisher</robot_param_node>
-                <parameters>$(find swing_drone)/config/drone_controller.yaml</parameters>
-            </plugin>
-        </gazebo>
     </xacro:macro>
 </robot>

File: src/swing_drone/urdf/robot_description.urdf.xacro (robot description, xacro)
@@ -3,5 +3,4 @@
   <!-- Dummy map link as root to avoid KDL parser warning -->
   <link name="map">
-    <!-- No inertia for dummy root link -->
   </link>
   <!-- Fixed joint connecting map to base_link -->
@@ -67,13 +66,4 @@
       </geometry>
     </visual>
-    <collision>
-      <origin
-        xyz="0 0 0"
-        rpy="0 0 0" />
-      <geometry>
-        <box
-          size="0.01 0.01 0.01" />
-      </geometry>
-    </collision>
   </link>
   <joint
@@ -85,8 +75,8 @@
       link="imu_link" />
     <origin
-      xyz="0 0 0"
+      xyz="0 0 0.01"
       rpy="0 0 0" />
     <axis
-      xyz="0 0 1" />
+      xyz="0 0 0" />
   </joint>
   <link

File: src/swing_drone/urdf/robot_gazebo.urdf.xacro (robot description, xacro)
@@ -7,121 +7,3 @@
         </plugin>
     </gazebo>
-    <gazebo>
-        <plugin name='ignition::gazebo::systems::Physics' filename='ignition-gazebo-physics-system'/>
-        <plugin name='ignition::gazebo::systems::UserCommands' filename='ignition-gazebo-user-commands-system'/>
-        <plugin name='ignition::gazebo::systems::SceneBroadcaster' filename='ignition-gazebo-scene-broadcaster-system'/>
-        <plugin filename="ignition-gazebo-sensors-system" name="ignition::gazebo::systems::Sensors"/>
-    </gazebo>
-  <gazebo reference="base_link">
-    <material>Gazebo/Blue</material>
-    <mu1>0.1</mu1>
-    <mu2>0.1</mu2>
-    <kp>1000000.0</kp>
-    <kd>1.0</kd>
-    <selfCollide>true</selfCollide>
-  </gazebo>
-  <gazebo reference="imu_link">
-    <material>Gazebo/Green</material>
-    <mu1>0.1</mu1>
-    <mu2>0.1</mu2>
-    <kp>1000000.0</kp>
-    <kd>1.0</kd>
-    <selfCollide>true</selfCollide>
-  </gazebo>
-  <gazebo reference="fr_link">
-    <material>Gazebo/Grey</material>
-    <mu1>0.1</mu1>
-    <mu2>0.1</mu2>
-    <kp>1000000.0</kp>
-    <kd>1.0</kd>
-    <selfCollide>true</selfCollide>
-  </gazebo>
-  <gazebo reference="br_link">
-    <material>Gazebo/Grey</material>
-    <mu1>0.1</mu1>
-    <mu2>0.1</mu2>
-    <kp>1000000.0</kp>
-    <kd>1.0</kd>
-    <selfCollide>true</selfCollide>
-  </gazebo>
-  <gazebo reference="fl_link">
-    <material>Gazebo/Grey</material>
-    <mu1>0.1</mu1>
-    <mu2>0.1</mu2>
-    <kp>1000000.0</kp>
-    <kd>1.0</kd>
-    <selfCollide>true</selfCollide>
-  </gazebo>
-  <gazebo reference="bl_link">
-    <material>Gazebo/Grey</material>
-    <mu1>0.1</mu1>
-    <mu2>0.1</mu2>
-    <kp>1000000.0</kp>
-    <kd>1.0</kd>
-    <selfCollide>true</selfCollide>
-  </gazebo>
-  <gazebo reference="A_prop_link">
-    <material>Gazebo/Red</material>
-    <mu1>0.1</mu1>
-    <mu2>0.1</mu2>
-    <kp>1000000.0</kp>
-    <kd>1.0</kd>
-    <selfCollide>false</selfCollide>
-  </gazebo>
-  <gazebo reference="B_prop_link">
-    <material>Gazebo/Grey</material>
-    <mu1>0.1</mu1>
-    <mu2>0.1</mu2>
-    <kp>1000000.0</kp>
-    <kd>1.0</kd>
-    <selfCollide>false</selfCollide>
-  </gazebo>
-  <gazebo reference="C_prop_link">
-    <material>Gazebo/Grey</material>
-    <mu1>0.1</mu1>
-    <mu2>0.1</mu2>
-    <kp>1000000.0</kp>
-    <kd>1.0</kd>
-    <selfCollide>false</selfCollide>
-  </gazebo>
-  <gazebo reference="D_prop_link">
-    <material>Gazebo/Grey</material>
-    <mu1>0.1</mu1>
-    <mu2>0.1</mu2>
-    <kp>1000000.0</kp>
-    <kd>1.0</kd>
-    <selfCollide>false</selfCollide>
-  </gazebo>
-  <gazebo reference="E_prop_link">
-    <material>Gazebo/Grey</material>
-    <mu1>0.1</mu1>
-    <mu2>0.1</mu2>
-    <kp>1000000.0</kp>
-    <kd>1.0</kd>
-    <selfCollide>false</selfCollide>
-  </gazebo>
-  <gazebo reference="F_prop_link">
-    <material>Gazebo/Grey</material>
-    <mu1>0.1</mu1>
-    <mu2>0.1</mu2>
-    <kp>1000000.0</kp>
-    <kd>1.0</kd>
-    <selfCollide>false</selfCollide>
-  </gazebo>
-  <gazebo reference="G_prop_link">
-    <material>Gazebo/Grey</material>
-    <mu1>0.1</mu1>
-    <mu2>0.1</mu2>
-    <kp>1000000.0</kp>
-    <kd>1.0</kd>
-    <selfCollide>false</selfCollide>
-  </gazebo>
-  <gazebo reference="H_prop_link">
-    <material>Gazebo/Red</material>
-    <mu1>0.1</mu1>
-    <mu2>0.1</mu2>
-    <kp>1000000.0</kp>
-    <kd>1.0</kd>
-    <selfCollide>false</selfCollide>
-  </gazebo>
 </robot>

Commit message: fix try add some lift drag and etc

File: src/swing_drone/urdf/robot_control.urdf.xacro (robot description, xacro)
@@ -7,5 +7,5 @@
             </hardware>
             <joint name="A_prop_joint">
-                <command_interface name="effort"></command_interface>
+                <command_interface name="velocity"></command_interface>
                 <state_interface name="position"/>
                 <state_interface name="velocity"/>
@@ -13,5 +13,5 @@
             </joint>
             <joint name="B_prop_joint">
-                <command_interface name="effort"></command_interface>
+                <command_interface name="velocity"></command_interface>
                 <state_interface name="position"/>
                 <state_interface name="velocity"/>
@@ -19,5 +19,5 @@
             </joint>
             <joint name="C_prop_joint">
-                <command_interface name="effort"></command_interface>
+                <command_interface name="velocity"></command_interface>
                 <state_interface name="position"/>
                 <state_interface name="velocity"/>
@@ -25,5 +25,5 @@
             </joint>
             <joint name="D_prop_joint">
-                <command_interface name="effort"></command_interface>
+                <command_interface name="velocity"></command_interface>
                 <state_interface name="position"/>
                 <state_interface name="velocity"/>
@@ -31,5 +31,5 @@
             </joint>
             <joint name="E_prop_joint">
-                <command_interface name="effort"></command_interface>
+                <command_interface name="velocity"></command_interface>
                 <state_interface name="position"/>
                 <state_interface name="velocity"/>
@@ -37,5 +37,5 @@
             </joint>
             <joint name="F_prop_joint">
-                <command_interface name="effort"></command_interface>
+                <command_interface name="velocity"></command_interface>
                 <state_interface name="position"/>
                 <state_interface name="velocity"/>
@@ -43,5 +43,5 @@
             </joint>
             <joint name="G_prop_joint">
-                <command_interface name="effort"></command_interface>
+                <command_interface name="velocity"></command_interface>
                 <state_interface name="position"/>
                 <state_interface name="velocity"/>
@@ -49,5 +49,5 @@
             </joint>
             <joint name="H_prop_joint">
-                <command_interface name="effort"></command_interface>
+                <command_interface name="velocity"></command_interface>
                 <state_interface name="position"/>
                 <state_interface name="velocity"/>

File: src/swing_drone/urdf/robot_description.urdf.xacro (robot description, xacro)
@@ -168,6 +168,5 @@
         rpy="0 0 0" />
       <geometry>
-        <mesh
-          filename="package://swing_drone/meshes/CCW_prop.STL" />
+        <cylinder radius="0.0635" length="0.01" />
       </geometry>
     </collision>
@@ -221,6 +220,5 @@
         rpy="0 0 0" />
       <geometry>
-        <mesh
-          filename="package://swing_drone/meshes/CW_prop.STL" />
+        <cylinder radius="0.0635" length="0.01" />
       </geometry>
     </collision>
@@ -327,6 +325,5 @@
         rpy="0 0 0" />
       <geometry>
-        <mesh
-          filename="package://swing_drone/meshes/CCW_prop.STL" />
+        <cylinder radius="0.0635" length="0.01" />
       </geometry>
     </collision>
@@ -380,6 +377,5 @@
         rpy="0 0 0" />
       <geometry>
-        <mesh
-          filename="package://swing_drone/meshes/CW_prop.STL" />
+        <cylinder radius="0.0635" length="0.01" />
       </geometry>
     </collision>
@@ -486,6 +482,5 @@
         rpy="0 0 0" />
       <geometry>
-        <mesh
-          filename="package://swing_drone/meshes/CCW_prop.STL" />
+        <cylinder radius="0.0635" length="0.01" />
       </geometry>
     </collision>
@@ -539,6 +534,5 @@
         rpy="0 0 0" />
       <geometry>
-        <mesh
-          filename="package://swing_drone/meshes/CW_prop.STL" />
+        <cylinder radius="0.0635" length="0.01" />
       </geometry>
     </collision>
@@ -645,6 +639,5 @@
         rpy="0 0 0" />
       <geometry>
-        <mesh
-          filename="package://swing_drone/meshes/CCW_prop.STL" />
+        <cylinder radius="0.0635" length="0.01" />
       </geometry>
     </collision>
@@ -698,6 +691,5 @@
         rpy="0 0 0" />
       <geometry>
-        <mesh
-          filename="package://swing_drone/meshes/CW_prop.STL" />
+        <cylinder radius="0.0635" length="0.01" />
       </geometry>
     </collision>

File: src/swing_drone/urdf/robot_gazebo.urdf.xacro (robot description, xacro)
@@ -1,4 +1,7 @@
 <?xml version="1.0"?>
-<robot xmlns:xacro="http://www.ros.org/wiki/xacro" name="swing_drone">
+<!-- Gazebo-specific configurations for swing_drone -->
+<robot xmlns:xacro="http://www.ros.org/wiki/xacro">
+    <!-- Removed the ign_ros2_control plugin to avoid conflict with PX4 MAVLink control -->
+    <!--
     <gazebo>
         <plugin filename="ign_ros2_control-system" name="ign_ros2_control::IgnitionROS2ControlPlugin">
@@ -7,4 +10,94 @@
         </plugin>
     </gazebo>
+    -->
+    <!-- Lift and Drag plugins for each propeller -->
+    <gazebo>
+        <plugin filename="libignition-gazebo-lift-drag-system.so" name="ignition::gazebo::systems::LiftDrag">
+            <link_name>A_prop_link</link_name>
+            <air_density>1.2041</air_density>
+            <center_pressure>0 0 0</center_pressure>
+            <direction>0 0 1</direction>
+            <upward>0 1 0</upward>
+            <area>0.0083</area>
+            <coefficient>1.3</coefficient>
+        </plugin>
+    </gazebo>
+    <gazebo>
+        <plugin filename="libignition-gazebo-lift-drag-system.so" name="ignition::gazebo::systems::LiftDrag">
+            <link_name>B_prop_link</link_name>
+            <air_density>1.2041</air_density>
+            <center_pressure>0 0 0</center_pressure>
+            <direction>0 0 1</direction>
+            <upward>0 1 0</upward>
+            <area>0.0083</area>
+            <coefficient>1.3</coefficient>
+        </plugin>
+    </gazebo>
+    <gazebo>
+        <plugin filename="libignition-gazebo-lift-drag-system.so" name="ignition::gazebo::systems::LiftDrag">
+            <link_name>C_prop_link</link_name>
+            <air_density>1.2041</air_density>
+            <center_pressure>0 0 0</center_pressure>
+            <direction>0 0 1</direction>
+            <upward>0 1 0</upward>
+            <area>0.0083</area>
+            <coefficient>1.3</coefficient>
+        </plugin>
+    </gazebo>
+    <gazebo>
+        <plugin filename="libignition-gazebo-lift-drag-system.so" name="ignition::gazebo::systems::LiftDrag">
+            <link_name>D_prop_link</link_name>
+            <air_density>1.2041</air_density>
+            <center_pressure>0 0 0</center_pressure>
+            <direction>0 0 1</direction>
+            <upward>0 1 0</upward>
+            <area>0.0083</area>
+            <coefficient>1.3</coefficient>
+        </plugin>
+    </gazebo>
+    <gazebo>
+        <plugin filename="libignition-gazebo-lift-drag-system.so" name="ignition::gazebo::systems::LiftDrag">
+            <link_name>E_prop_link</link_name>
+            <air_density>1.2041</air_density>
+            <center_pressure>0 0 0</center_pressure>
+            <direction>0 0 1</direction>
+            <upward>0 1 0</upward>
+            <area>0.0083</area>
+            <coefficient>1.3</coefficient>
+        </plugin>
+    </gazebo>
+    <gazebo>
+        <plugin filename="libignition-gazebo-lift-drag-system.so" name="ignition::gazebo::systems::LiftDrag">
+            <link_name>F_prop_link</link_name>
+            <air_density>1.2041</air_density>
+            <center_pressure>0 0 0</center_pressure>
+            <direction>0 0 1</direction>
+            <upward>0 1 0</upward>
+            <area>0.0083</area>
+            <coefficient>1.3</coefficient>
+        </plugin>
+    </gazebo>
+    <gazebo>
+        <plugin filename="libignition-gazebo-lift-drag-system.so" name="ignition::gazebo::systems::LiftDrag">
+            <link_name>G_prop_link</link_name>
+            <air_density>1.2041</air_density>
+            <center_pressure>0 0 0</center_pressure>
+            <direction>0 0 1</direction>
+            <upward>0 1 0</upward>
+            <area>0.0083</area>
+            <coefficient>1.3</coefficient>
+        </plugin>
+    </gazebo>
+    <gazebo>
+        <plugin filename="libignition-gazebo-lift-drag-system.so" name="ignition::gazebo::systems::LiftDrag">
+            <link_name>H_prop_link</link_name>
+            <air_density>1.2041</air_density>
+            <center_pressure>0 0 0</center_pressure>
+            <direction>0 0 1</direction>
+            <upward>0 1 0</upward>
+            <area>0.0083</area>
+            <coefficient>1.3</coefficient>
+        </plugin>
+    </gazebo>
     <gazebo reference="base_link">
         <mu1>1.0</mu1>
@@ -15,5 +108,5 @@
         <dampingFactor>0.001</dampingFactor>
     </gazebo>
-    <gazebo reference="fr_link  ">
+    <gazebo reference="fr_link">
         <mu1>1.0</mu1>
         <mu2>1.0</mu2>
@@ -112,9 +205,3 @@
     </sensor>
   </gazebo>
-<gazebo>
-  <plugin name="joint_wrench_plugin" filename="libjoint_wrench_plugin.so">
-    <joint_name>A_prop_joint</joint_name>
-    <topic_name>/Drone/A_prop_joint/wrench</topic_name>
-  </plugin>
-</gazebo>
 </robot>
